File: edge-key-seventeen.kicad_pcb (KiCad board)
At the start: 2 copper layers, 112.7 x 99.7 mm, 78 parts, among them J1 USB_B_Micro, J2 AVR-ISP-6, SW1 Rotary_Encoder_Switch, SW2 Rotary_Encoder_Switch, U1 ATMEGA32U4, Y1 16 MHz

Commit message: update.
Parts:
- removed REF**: W-Logo, myFootprints:W-Logo
- removed the Ref** at (195.1, 87.4) (x2)
- added D30: LED, LED_THT:LED_D5.0mm, F.Cu at (146.8, 55.4)
- added R10: 330, Resistor_SMD:R_0805_2012Metric_Pad1.20x1.40mm_HandSolder, B.Cu at (157.5, 58.4)
- added R6: 5.1k, Resistor_SMD:R_0603_1608Metric_Pad0.98x0.95mm_HandSolder, B.Cu at (132.8, 105.2)
- added R8: 5.1k, Resistor_SMD:R_0603_1608Metric_Pad0.98x0.95mm_HandSolder, B.Cu at (126.2, 109.6)
- added R9: 330, Resistor_SMD:R_0805_2012Metric_Pad1.20x1.40mm_HandSolder, F.Cu at (152.4, 56.4)
- added Ref**: Val**, logo:keyboard-bit, F.Cu at (191.3, 86.1)
- added Ref**: Val**, logo:keyboard-bit, B.Cu at (191.3, 86.1)
- C10, C5, C6, C7, C8: footprint Capacitor_SMD:C_0805_2012Metric_Pad1.15x1.40mm_HandSolder -> Capacitor_SMD:C_0603_1608Metric_Pad1.08x0.95mm_HandSolder
- D8: footprint myFootprints:TO-253-4_HandSolder -> Package_TO_SOT_SMD:SOT-143_Handsoldering
- J1: footprint Connector_USB:USB_Micro-B_Amphenol_10103594-0001LF_Horizontal -> Connector_USB:USB_C_Receptacle_GCT_USB4085
- MX1: footprint MX_Only:MXOnly-1U-NoLED -> MX_Only:MXOnly-1U
- R1: footprint Resistor_SMD:R_0805_2012Metric_Pad1.15x1.40mm_HandSolder -> Resistor_SMD:R_0603_1608Metric_Pad0.98x0.95mm_HandSolder; moved to F.Cu
- R2, R3, R7: footprint Resistor_SMD:R_0805_2012Metric_Pad1.15x1.40mm_HandSolder -> Resistor_SMD:R_0603_1608Metric_Pad0.98x0.95mm_HandSolder
- R5: footprint Resistor_SMD:R_0805_2012Metric_Pad1.15x1.40mm_HandSolder -> Resistor_SMD:R_0805_2012Metric_Pad1.20x1.40mm_HandSolder
- S1: footprint SparkFun-Switches:TACTILE_SWITCH_SMD_5.2MM -> myFootprints:SW_KSR223GLFG
- Y1: footprint Crystal:Crystal_HC49-U_Vertical -> Crystal:Crystal_SMD_3225-4Pin_3.2x2.5mm_HandSoldering
- moved R7 11.1 mm to (127.0, 100.8)
- moved C10 10.9 mm to (125.5, 100.8)
- moved C3 5.73 mm to (133.3, 112.8)
- moved R2 3.75 mm to (136.9, 106.9), turned to 0 degrees
- moved J1 3.64 mm to (130.0, 105.5)
- moved R1 3.60 mm to (147.1, 134.6)
- moved Y1 3.09 mm to (146.6, 130.2), turned to -45 degrees
- moved D8 2.34 mm to (133.3, 108.5)
- moved S1 1.05 mm to (134.9, 125.0)
- moved R3 1.02 mm to (136.9, 110.0), turned to 0 degrees
- moved F1 0.46 mm to (132.3, 101.3)
Connections:
- D26 pad 4: (no net) -> unconnected-(D26-Pad4)
- D8 pad 1: Net-(C10-Pad1) -> GND
- D8 pad 2: /D+ -> /D-
- D8 pad 3: /D- -> /D+
- J2 pad 5: ~RESET -> ~{RESET}
- R4 pad 1: ~RESET -> ~{RESET}
- S1 pad 1: ~RESET -> ~{RESET}
- S1 pad 2: ~RESET -> GND
- U1 pad 1: (no net) -> unconnected-(U1-Pad1)
- U1 pad 13: ~RESET -> ~{RESET}
- U1 pad 18: (no net) -> unconnected-(U1-Pad18)
- U1 pad 19: (no net) -> unconnected-(U1-Pad19)
- U1 pad 26: (no net) -> unconnected-(U1-Pad26)
- U1 pad 27: (no net) -> unconnected-(U1-Pad27)
- U1 pad 36: (no net) -> PF7
- U1 pad 42: (no net) -> unconnected-(U1-Pad42)
- U1 pad 8: (no net) -> unconnected-(U1-Pad8)
- Y1 pad 2: OSC2 -> GND
Routing:
- net PF7: track 0.00 -> 60.2 mm, vias 0 -> 3
- net ~{RESET}: track 0.00 -> 21.1 mm
- net ~RESET: track 20.7 -> 0.00 mm, vias 2 -> 0
- net VCC: track 50.8 -> 41.7 mm
- net Net-(MX1-Pad3): track 0.00 -> 4.68 mm
- net /ID+: track 6.44 -> 10.7 mm
- net OSC2: track 10.1 -> 14.2 mm
- net OSC1: track 10.1 -> 13.9 mm
- net GND: track 25.7 -> 22.1 mm, vias 22 -> 11
- net /VUSB: track 3.18 -> 0.00 mm
- net /CC1: track 0.00 -> 3.11 mm
- net Net-(D30-Pad2): track 0.00 -> 3.05 mm
- net PF0: track 50.0 -> 47.1 mm
- net Net-(C10-Pad1): track 21.8 -> 19.5 mm
- net PB6: track 131.9 -> 133.7 mm
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- removed copper zone on F.Cu, net Net-(C10-Pad1)
Other:
- net class Default removed
- net class VCC removed
- board text added: "Col: PF0, PD4, PD5, PD3, PD2 Row: PB6, PC7, PC6. PB5, PB4 Encoders: PF5/PF6, PF1/PF4 Col -> Row Neopixel: PB7 LED: PF7"
- board text added: "Edge Key Seventeen Numeric Keypad v1.0 rev 2"
- board text removed: "Col: PF0, PD4, PD5, PD3, PD2 Row: PB6, PC7, PC6. PB5, PB4 Encoders: PF5/PF6, PF1/PF4 Col -> Row Neopixel: PB7"
- board text removed: "Edge Key Seventeen Numeric Keypad v1.0 rev 1"
- board text removed: "GND"
- board text removed: "MicroUSB"
- board text removed: "Vcc"
